File: pcb/ai_aurora.sch (EAGLE design)
At the start: 24 parts, among them IC1 ATTINY85-DIP, J1 1X02ST, J2 2X03, Q1 FQP30N06L

Commit message: gerbers
Parts:
- added M2, M3, PANEL+, PANEL-: 1X01-TERM-PANEL, Ai_Connectors:1X01-TERM-PANEL
- renumbered J1 to SOLAR-IN, J2 to ISP, S1 to RESET, S2 to SET
Connections:
- removed net N$2: D1.A, SOLAR-IN.1
- new net VPANEL: D1.A, PANEL+.1, SOLAR-IN.1
- net GND: now also PANEL-.1
- net MOSI/SET: now also SET.B@1
Changed lines of the file:
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@@
 <?xml version="1.0" encoding="utf-8"?>
 <!DOCTYPE eagle SYSTEM "eagle.dtd">
-<eagle version="7.1.0">
+<eagle version="6.5.0">
 <drawing>
 <settings>
@@
 <part name="C2" library="Ai_Passives" deviceset="CAP" device="025X050"/>
 <part name="D1" library="Ai_DiscreteSemis" deviceset="DIODE" device="TH-1N914"/>
-<part name="J1" library="Ai_Connectors" deviceset="1X02" device="ST"/>
-<part name="J2" library="Ai_Connectors" deviceset="2X03" device=""/>
+<part name="SOLAR-IN" library="Ai_Connectors" deviceset="1X02" device="ST"/>
+<part name="ISP" library="Ai_Connectors" deviceset="2X03" device=""/>
 <part name="U$1" library="Ai_Power" deviceset="VIN" device=""/>
 <part name="GND1" library="Ai_Power" deviceset="GND" device=""/>
@@
 <part name="R1" library="Ai_Passives" deviceset="RES" device="AXIAL-0.4" value="10K"/>
 <part name="GND9" library="Ai_Power" deviceset="GND" device=""/>
-<part name="S1" library="Ai_Electromechanical" deviceset="SW-SPST" device="TH06X06"/>
+<part name="RESET" library="Ai_Electromechanical" deviceset="SW-SPST" device="TH06X06"/>
 <part name="U$6" library="Ai_Power" deviceset="VBAT" device=""/>
 <part name="VR1" library="Ai_Passives" deviceset="POT" device="05X05" value="1M"/>
@@
 <part name="U$8" library="Ai_Power" deviceset="VBAT" device=""/>
 <part name="GND6" library="Ai_Power" deviceset="GND" device=""/>
-<part name="S2" library="Ai_Electromechanical" deviceset="SW-SPST" device="TH06X06"/>
+<part name="SET" library="Ai_Electromechanical" deviceset="SW-SPST" device="TH06X06"/>
 <part name="R3" library="Ai_Passives" deviceset="RES" device="AXIAL-0.4" value="10K"/>
 <part name="GND7" library="Ai_Power" deviceset="GND" device=""/>
 <part name="R4" library="Ai_Passives" deviceset="RES" device="AXIAL-0.4" value="100K"/>
+<part name="PANEL+" library="Ai_Connectors" deviceset="1X01-TERM" device="-PANEL"/>
+<part name="PANEL-" library="Ai_Connectors" deviceset="1X01-TERM" device="-PANEL"/>
+<part name="U$11" library="Ai_Power" deviceset="VPANEL" device=""/>
+<part name="U$12" library="Ai_Power" deviceset="VPANEL" device=""/>
+<part name="GND8" library="Ai_Power" deviceset="GND" device=""/>
+<part name="M2" library="Ai_Connectors" deviceset="1X01-TERM" device="-PANEL"/>
+<part name="M3" library="Ai_Connectors" deviceset="1X01-TERM" device="-PANEL"/>
 </parts>
 <sheets>
@@
 <instance part="C2" gate="G$1" x="240.03" y="118.11"/>
 <instance part="D1" gate="G$1" x="30.48" y="115.57"/>
-<instance part="J1" gate="G$1" x="20.32" y="113.03" rot="MR180"/>
-<instance part="J2" gate="G$1" x="135.89" y="121.92" rot="R180"/>
+<instance part="SOLAR-IN" gate="G$1" x="20.32" y="113.03" rot="MR180"/>
+<instance part="ISP" gate="G$1" x="135.89" y="121.92" rot="R180"/>
 <instance part="U$1" gate="G$1" x="35.56" y="118.11"/>
 <instance part="GND1" gate="GND" x="27.94" y="107.95"/>
@@
 <instance part="R1" gate="G$1" x="151.13" y="77.47" rot="R90"/>
 <instance part="GND9" gate="GND" x="151.13" y="68.58"/>
-<instance part="S1" gate="G$1" x="151.13" y="88.9" rot="MR270"/>
+<instance part="RESET" gate="G$1" x="151.13" y="88.9" rot="MR270"/>
 <instance part="U$6" gate="G$1" x="146.05" y="127"/>
 <instance part="VR1" gate="G$1" x="87.63" y="120.65" rot="R180"/>
@@
 <instance part="U$8" gate="G$1" x="191.77" y="87.63"/>
 <instance part="GND6" gate="GND" x="191.77" y="58.42"/>
-<instance part="S2" gate="G$1" x="92.71" y="74.93"/>
+<instance part="SET" gate="G$1" x="92.71" y="74.93"/>
 <instance part="R3" gate="G$1" x="85.09" y="67.31" rot="R90"/>
 <instance part="GND7" gate="GND" x="85.09" y="58.42"/>
 <instance part="R4" gate="G$1" x="182.88" y="68.58" rot="R90"/>
+<instance part="PANEL+" gate="G$1" x="132.08" y="46.99"/>
+<instance part="PANEL-" gate="G$1" x="142.24" y="46.99"/>
+<instance part="U$11" gate="G$1" x="26.67" y="118.11"/>
+<instance part="U$12" gate="G$1" x="132.08" y="52.07"/>
+<instance part="GND8" gate="GND" x="142.24" y="40.64"/>
+<instance part="M2" gate="G$1" x="166.37" y="44.45"/>
+<instance part="M3" gate="G$1" x="172.72" y="44.45"/>
 </instances>
 <busses>
@@
 <wire x1="27.94" y1="113.03" x2="27.94" y2="110.49" width="0.1524" layer="91"/>
 <pinref part="GND1" gate="GND" pin="GND"/>
-<pinref part="J1" gate="G$1" pin="2"/>
+<pinref part="SOLAR-IN" gate="G$1" pin="2"/>
 <wire x1="25.4" y1="113.03" x2="27.94" y2="113.03" width="0.1524" layer="91"/>
 </segment>
@@
 </segment>
 <segment>
-<pinref part="J2" gate="G$1" pin="6"/>
+<pinref part="ISP" gate="G$1" pin="6"/>
 <wire x1="143.51" y1="119.38" x2="146.05" y2="119.38" width="0.1524" layer="91"/>
 <pinref part="GND4" gate="GND" pin="GND"/>
@@
 <wire x1="85.09" y1="60.96" x2="85.09" y2="62.23" width="0.1524" layer="91"/>
 </segment>
+<segment>
+<pinref part="GND8" gate="GND" pin="GND"/>
+<pinref part="PANEL-" gate="G$1" pin="1"/>
+<wire x1="142.24" y1="43.18" x2="142.24" y2="46.99" width="0.1524" layer="91"/>
+</segment>
 </net>
 <net name="VBAT" class="0">
@@
 </segment>
 <segment>
-<pinref part="J2" gate="G$1" pin="2"/>
+<pinref part="ISP" gate="G$1" pin="2"/>
 <wire x1="143.51" y1="124.46" x2="146.05" y2="124.46" width="0.1524" layer="91"/>
 <pinref part="U$6" gate="G$1" pin="VBAT"/>
@@
 <net name="MISO/LDR" class="0">
 <segment>
-<pinref part="J2" gate="G$1" pin="1"/>
+<pinref part="ISP" gate="G$1" pin="1"/>
 <wire x1="128.27" y1="124.46" x2="125.73" y2="124.46" width="0.1524" layer="91"/>
 <label x="125.73" y="124.46" size="1.27" layer="95" font="vector" ratio="10" rot="R180" xref="yes"/>
@@
 <net name="SCK/BATT" class="0">
 <segment>
-<pinref part="J2" gate="G$1" pin="3"/>
+<pinref part="ISP" gate="G$1" pin="3"/>
 <wire x1="128.27" y1="121.92" x2="125.73" y2="121.92" width="0.1524" layer="91"/>
 <label x="125.73" y="121.92" size="1.27" layer="95" font="vector" ratio="10" rot="R180" xref="yes"/>
@@
 <net name="RST" class="0">
 <segment>
-<pinref part="J2" gate="G$1" pin="5"/>
+<pinref part="ISP" gate="G$1" pin="5"/>
 <label x="125.73" y="119.38" size="1.27" layer="95" font="vector" ratio="10" rot="R180" xref="yes"/>
 <wire x1="128.27" y1="119.38" x2="125.73" y2="119.38" width="0.1524" layer="91"/>
@@
 <wire x1="149.86" y1="95.25" x2="151.13" y2="95.25" width="0.1524" layer="91"/>
 <wire x1="151.13" y1="95.25" x2="154.94" y2="95.25" width="0.1524" layer="91"/>
-<pinref part="S1" gate="G$1" pin="A@1"/>
+<pinref part="RESET" gate="G$1" pin="A@1"/>
 <wire x1="151.13" y1="95.25" x2="151.13" y2="93.98" width="0.1524" layer="91"/>
 <junction x="151.13" y="95.25"/>
@@
 <net name="MOSI/SET" class="0">
 <segment>
-<pinref part="J2" gate="G$1" pin="4"/>
+<pinref part="ISP" gate="G$1" pin="4"/>
 <wire x1="143.51" y1="121.92" x2="146.05" y2="121.92" width="0.1524" layer="91"/>
 <label x="146.05" y="121.92" size="1.27" layer="95" font="vector" ratio="10" xref="yes"/>
@@
 <wire x1="97.79" y1="74.93" x2="100.33" y2="74.93" width="0.1524" layer="91"/>
 <label x="100.33" y="74.93" size="1.27" layer="95" font="vector" ratio="10" xref="yes"/>
+<pinref part="SET" gate="G$1" pin="B@1"/>
 </segment>
 </net>
@@
 <pinref part="BAT1" gate="G$1" pin="+"/>
 <wire x1="48.26" y1="115.57" x2="50.8" y2="115.57" width="0.1524" layer="91"/>
-</segment>
-</net>
-<net name="N$2" class="0">
-<segment>
-<pinref part="J1" gate="G$1" pin="1"/>
-<pinref part="D1" gate="G$1" pin="A"/>
-<wire x1="25.4" y1="115.57" x2="27.94" y2="115.57" width="0.1524" layer="91"/>
 </segment>
 </net>
@@
 <net name="N$3" class="0">
 <segment>
-<pinref part="S1" gate="G$1" pin="B@1"/>
+<pinref part="RESET" gate="G$1" pin="B@1"/>
 <pinref part="R1" gate="G$1" pin="2"/>
 <wire x1="151.13" y1="83.82" x2="151.13" y2="82.55" width="0.1524" layer="91"/>
@@
 <pinref part="R3" gate="G$1" pin="2"/>
 <wire x1="85.09" y1="72.39" x2="85.09" y2="74.93" width="0.1524" layer="91"/>
-<pinref part="S2" gate="G$1" pin="A@1"/>
+<pinref part="SET" gate="G$1" pin="A@1"/>
 <wire x1="85.09" y1="74.93" x2="87.63" y2="74.93" width="0.1524" layer="91"/>
 </segment>
 </net>
+<net name="VPANEL" class="0">
+<segment>
+<pinref part="SOLAR-IN" gate="G$1" pin="1"/>
+<pinref part="D1" gate="G$1" pin="A"/>
+<wire x1="25.4" y1="115.57" x2="26.67" y2="115.57" width="0.1524" layer="91"/>
+<pinref part="U$11" gate="G$1" pin="VPANEL"/>
+<wire x1="26.67" y1="115.57" x2="27.94" y2="115.57" width="0.1524" layer="91"/>
+<wire x1="26.67" y1="118.11" x2="26.67" y2="115.57" width="0.1524" layer="91"/>
+<junction x="26.67" y="115.57"/>
+</segment>
+<segment>
+<pinref part="PANEL+" gate="G$1" pin="1"/>
+<pinref part="U$12" gate="G$1" pin="VPANEL"/>
+<wire x1="132.08" y1="46.99" x2="132.08" y2="52.07" width="0.1524" layer="91"/>
+</segment>
+</net>

Commit message: updated libraries
Parts:
- BAT1, BAT2: value (none) -> CR123A
- C1, C2: value (none) -> 0.1uF
Connections:
- removed net +: C1.1, C2.1, LED1.VDD, LED2.VDD
- net VBAT: now also C1.1, C2.1, LED1.VDD, LED2.VDD
Other:
- moved on the sheet: C2, M2, M3
Changed lines of the file:
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@@
 <layer number="223" name="223bmp" color="24" fill="1" visible="no" active="no"/>
 <layer number="224" name="224bmp" color="25" fill="1" visible="no" active="no"/>
+<layer number="225" name="225bmp" color="7" fill="1" visible="no" active="yes"/>
+<layer number="226" name="226bmp" color="7" fill="1" visible="no" active="yes"/>
+<layer number="227" name="227bmp" color="7" fill="1" visible="no" active="yes"/>
+<layer number="228" name="228bmp" color="7" fill="1" visible="no" active="yes"/>
+<layer number="230" name="230bmp" color="7" fill="1" visible="no" active="yes"/>
 <layer number="248" name="Housing" color="7" fill="1" visible="yes" active="yes"/>
 <layer number="249" name="Edge" color="7" fill="1" visible="yes" active="yes"/>
@@
 <part name="GND5" library="Ai_Power" deviceset="GND" device=""/>
 <part name="U$2" library="Ai_Power" deviceset="VBAT" device=""/>
-<part name="BAT1" library="Ai_Electromechanical" deviceset="BATTERY-HOLDER" device="CR123A"/>
-<part name="BAT2" library="Ai_Electromechanical" deviceset="BATTERY-HOLDER" device="CR123A"/>
-<part name="C1" library="Ai_Passives" deviceset="CAP" device="025X050"/>
-<part name="C2" library="Ai_Passives" deviceset="CAP" device="025X050"/>
+<part name="BAT1" library="Ai_Electromechanical" deviceset="BATTERY-HOLDER" device="CR123A" value="CR123A"/>
+<part name="BAT2" library="Ai_Electromechanical" deviceset="BATTERY-HOLDER" device="CR123A" value="CR123A"/>
+<part name="C1" library="Ai_Passives" deviceset="CAP" device="025X050" value="0.1uF"/>
+<part name="C2" library="Ai_Passives" deviceset="CAP" device="025X050" value="0.1uF"/>
 <part name="D1" library="Ai_DiscreteSemis" deviceset="DIODE" device="TH-1N914"/>
 <part name="SOLAR-IN" library="Ai_Connectors" deviceset="1X02" device="ST"/>
@@
 <instance part="BAT2" gate="G$1" x="55.88" y="115.57" rot="R180"/>
 <instance part="C1" gate="G$1" x="232.41" y="118.11"/>
-<instance part="C2" gate="G$1" x="240.03" y="118.11"/>
+<instance part="C2" gate="G$1" x="241.3" y="118.11"/>
 <instance part="D1" gate="G$1" x="30.48" y="115.57"/>
 <instance part="SOLAR-IN" gate="G$1" x="20.32" y="113.03" rot="MR180"/>
@@
 <instance part="U$12" gate="G$1" x="132.08" y="52.07"/>
 <instance part="GND8" gate="GND" x="142.24" y="40.64"/>
-<instance part="M2" gate="G$1" x="166.37" y="44.45"/>
-<instance part="M3" gate="G$1" x="172.72" y="44.45"/>
+<instance part="M2" gate="G$1" x="135.89" y="6.35"/>
+<instance part="M3" gate="G$1" x="142.24" y="6.35"/>
 </instances>
 <busses>
@@
 <wire x1="119.38" y1="107.95" x2="119.38" y2="110.49" width="0.1524" layer="91"/>
 </segment>
-</net>
-<net name="+" class="0">
 <segment>
 <pinref part="C1" gate="G$1" pin="1"/>
@@
 <segment>
 <pinref part="C2" gate="G$1" pin="1"/>
-<wire x1="240.03" y1="123.19" x2="240.03" y2="125.73" width="0.1524" layer="91"/>
-<label x="240.03" y="125.73" size="1.27" layer="95" font="vector" ratio="10" rot="R180" xref="yes"/>
+<wire x1="241.3" y1="123.19" x2="241.3" y2="125.73" width="0.1524" layer="91"/>
+<label x="241.3" y="125.73" size="1.27" layer="95" font="vector" ratio="10" rot="R180" xref="yes"/>
 </segment>
 <segment>
@@
 <segment>
 <pinref part="C2" gate="G$1" pin="2"/>
-<wire x1="240.03" y1="107.95" x2="240.03" y2="113.03" width="0.1524" layer="91"/>
-<label x="240.03" y="107.95" size="1.27" layer="95" font="vector" ratio="10" xref="yes"/>
+<wire x1="241.3" y1="107.95" x2="241.3" y2="113.03" width="0.1524" layer="91"/>
+<label x="241.3" y="107.95" size="1.27" layer="95" font="vector" ratio="10" xref="yes"/>
 </segment>
 <segment>
@@
 </sheet>
 </sheets>
+<errors>
+</errors>
 </schematic>
 </drawing>

Commit message: minor update to schematic
Parts:
- BAT1, BAT2: value CR123A -> (none)
- C1, C2: value 0.1uF -> (none)
Connections:
- new net +: C1.1, C2.1, LED1.VDD, LED2.VDD
- net VBAT: no longer C1.1, C2.1, LED1.VDD, LED2.VDD
Other:
- moved on the sheet: C2, M2, M3
Changed lines of the file:
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@@
 <part name="GND5" library="Ai_Power" deviceset="GND" device=""/>
 <part name="U$2" library="Ai_Power" deviceset="VBAT" device=""/>
-<part name="BAT1" library="Ai_Electromechanical" deviceset="BATTERY-HOLDER" device="CR123A" value="CR123A"/>
-<part name="BAT2" library="Ai_Electromechanical" deviceset="BATTERY-HOLDER" device="CR123A" value="CR123A"/>
-<part name="C1" library="Ai_Passives" deviceset="CAP" device="025X050" value="0.1uF"/>
-<part name="C2" library="Ai_Passives" deviceset="CAP" device="025X050" value="0.1uF"/>
+<part name="BAT1" library="Ai_Electromechanical" deviceset="BATTERY-HOLDER" device="CR123A"/>
+<part name="BAT2" library="Ai_Electromechanical" deviceset="BATTERY-HOLDER" device="CR123A"/>
+<part name="C1" library="Ai_Passives" deviceset="CAP" device="025X050"/>
+<part name="C2" library="Ai_Passives" deviceset="CAP" device="025X050"/>
 <part name="D1" library="Ai_DiscreteSemis" deviceset="DIODE" device="TH-1N914"/>
 <part name="SOLAR-IN" library="Ai_Connectors" deviceset="1X02" device="ST"/>
@@
 <instance part="BAT2" gate="G$1" x="55.88" y="115.57" rot="R180"/>
 <instance part="C1" gate="G$1" x="232.41" y="118.11"/>
-<instance part="C2" gate="G$1" x="241.3" y="118.11"/>
+<instance part="C2" gate="G$1" x="240.03" y="118.11"/>
 <instance part="D1" gate="G$1" x="30.48" y="115.57"/>
 <instance part="SOLAR-IN" gate="G$1" x="20.32" y="113.03" rot="MR180"/>
@@
 <instance part="U$12" gate="G$1" x="132.08" y="52.07"/>
 <instance part="GND8" gate="GND" x="142.24" y="40.64"/>
-<instance part="M2" gate="G$1" x="135.89" y="6.35"/>
-<instance part="M3" gate="G$1" x="142.24" y="6.35"/>
+<instance part="M2" gate="G$1" x="166.37" y="44.45"/>
+<instance part="M3" gate="G$1" x="172.72" y="44.45"/>
 </instances>
 <busses>
@@
 <wire x1="119.38" y1="107.95" x2="119.38" y2="110.49" width="0.1524" layer="91"/>
 </segment>
+</net>
+<net name="+" class="0">
 <segment>
 <pinref part="C1" gate="G$1" pin="1"/>
@@
 <segment>
 <pinref part="C2" gate="G$1" pin="1"/>
-<wire x1="241.3" y1="123.19" x2="241.3" y2="125.73" width="0.1524" layer="91"/>
-<label x="241.3" y="125.73" size="1.27" layer="95" font="vector" ratio="10" rot="R180" xref="yes"/>
+<wire x1="240.03" y1="123.19" x2="240.03" y2="125.73" width="0.1524" layer="91"/>
+<label x="240.03" y="125.73" size="1.27" layer="95" font="vector" ratio="10" rot="R180" xref="yes"/>
 </segment>
 <segment>
@@
 <segment>
 <pinref part="C2" gate="G$1" pin="2"/>
-<wire x1="241.3" y1="107.95" x2="241.3" y2="113.03" width="0.1524" layer="91"/>
-<label x="241.3" y="107.95" size="1.27" layer="95" font="vector" ratio="10" xref="yes"/>
+<wire x1="240.03" y1="107.95" x2="240.03" y2="113.03" width="0.1524" layer="91"/>
+<label x="240.03" y="107.95" size="1.27" layer="95" font="vector" ratio="10" xref="yes"/>
 </segment>
 <segment>
@@
 </sheet>
 </sheets>
-<errors>
-</errors>
 </schematic>
 </drawing>
